File: PCB/aux-PCB/aux-PCB.kicad_pcb (KiCad board)
At the start: 2 copper layers, 19.9 x 18.2 mm, 6 parts

Commit message: -Added custom silkscreen -Generated gerbers -Exported STEP files
Other:
- board text removed: "EN 03/2026"

Commit message: Updated PCB STEP file
Parts:
- R1, R4: value 430 -> 120; footprint Resistor_SMD:R_0201_0603Metric -> Resistor_SMD:R_0402_1005Metric
