File: PCB/aux-PCB/aux-PCB.kicad_pcb (KiCad board)
At the start: 2 copper layers, 19.9 x 18.2 mm, 6 parts

Commit message: -In progress porting code to LIS2DW12.
Other:
- outline, holes or cut-outs redrawn
Changed lines of the file:
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@@
+		(layer "Edge.Cuts")
+	)
+	(gr_circle
+		(center 141.8 87.6)
+		(end 142.5 87.6)
+		(stroke
+			(width 0.2)
+			(type solid)
+		)
+		(fill no)
 		(layer "Edge.Cuts")
 	)
@@
 		(layer "Edge.Cuts")
 	)
+	(gr_circle
+		(center 158.2 87.6)
+		(end 158.9 87.6)
+		(stroke
+			(width 0.2)
+			(type solid)
+		)
+		(fill no)
+		(layer "Edge.Cuts")
+	)
 	(gr_line
 		(start 158.313913 83.084536)
@@
 		)
 		(layer "Edge.Cuts")
+	)
+	(gr_circle
+		(center 141.8 87.6)
+		(end 142.9 87.6)
+		(stroke
+			(width 0.2)
+			(type solid)
+		)
+		(fill no)
+		(layer "F.Fab")
+	)
+	(gr_circle
+		(center 158.2 87.6)
+		(end 159.3 87.6)
+		(stroke
+			(width 0.2)
+			(type solid)
+		)
+		(fill no)
+		(layer "F.Fab")
 	)
 	(gr_poly
@@
 	)
 	(segment
+		(start 143.6 86.9)
+		(end 143 86.3)
+		(width 0.4)
+		(layer "F.Cu")
+		(net "/LED_K")
+	)
+	(segment
+		(start 143 86.3)
+		(end 143 85)
+		(width 0.4)
+		(layer "F.Cu")
+		(net "/LED_K")
+	)
+	(via
+		(at 143.6 86.9)
+		(size 0.6)
+		(drill 0.4)
+		(layers "F.Cu" "B.Cu")
+		(capping no)
+		(covering
+			(front no)
+			(back no)
+		)
+		(plugging
+			(front no)
+			(back no)
+		)
+		(filling no)
+		(net "/LED_K")
+	)
+	(segment
+		(start 144.342947 87.657053)
+		(end 144.342947 87.642947)
+		(width 0.4)
+		(layer "B.Cu")
+		(net "/LED_K")
+	)
+	(segment
+		(start 144.342947 87.642947)
+		(end 143.6 86.9)
+		(width 0.4)
+		(layer "B.Cu")
+		(net "/LED_K")
+	)
+	(segment
+		(start 155.657053 87.657053)
+		(end 144.342947 87.657053)
+		(width 0.4)
+		(layer "B.Cu")
+		(net "/LED_K")
+	)
+	(segment
 		(start 151 91)
 		(end 150 91)
@@
 	)
 	(segment
-		(start 143.6 86.9)
-		(end 143 86.3)
-		(width 0.4)
-		(layer "F.Cu")
-		(net "/LED_K")
-	)
-	(segment
-		(start 143 86.3)
-		(end 143 85)
-		(width 0.4)
-		(layer "F.Cu")
-		(net "/LED_K")
-	)
-	(via
-		(at 143.6 86.9)
-		(size 0.6)
-		(drill 0.4)
-		(layers "F.Cu" "B.Cu")
-		(capping no)
-		(covering
-			(front no)
-			(back no)
-		)
-		(plugging
-			(front no)
-			(back no)
-		)
-		(filling no)
-		(net "/LED_K")
-	)
-	(segment
-		(start 144.342947 87.657053)
-		(end 144.342947 87.642947)
+		(start 156.342947 88.342947)
+		(end 157.039376 89.039376)
 		(width 0.4)
 		(layer "B.Cu")
-		(net "/LED_K")
-	)
-	(segment
-		(start 144.342947 87.642947)
-		(end 143.6 86.9)
-		(width 0.4)
-		(layer "B.Cu")
-		(net "/LED_K")
-	)
-	(segment
-		(start 155.657053 87.657053)
-		(end 144.342947 87.657053)
-		(width 0.4)
-		(layer "B.Cu")
-		(net "/LED_K")
+		(net "Net-(D2-A)")
 	)
 	(segment
@@
 		(net "Net-(D1-A)")
 	)
-	(segment
-		(start 156.342947 88.342947)
-		(end 157.039376 89.039376)
-		(width 0.4)
-		(layer "B.Cu")
-		(net "Net-(D2-A)")
-	)
 	(group ""
