File: PCB/aux-PCB/aux-PCB.kicad_sch (KiCad schematic)
At the start: 6 parts

Commit message: Updated PCB STEP file
Parts:
- R1, R4: value 430 -> 120; footprint Resistor_SMD:R_0201_0603Metric -> Resistor_SMD:R_0402_1005Metric
