File: PCB/main-PCB/main-PCB.kicad_pcb (KiCad board)
At the start: 4 copper layers, 20 x 18.3 mm, 43 parts, among them Q1 SSM6J214FE, Q2 Q_NMOS_GSD, U1 LIS2DU12TR, U2 STM32U031K4Ux

Commit message: Add heartbeat LED PWM pattern and low-power sleep/wake cycle
- Drive the heart LED via TIM2 CH4 PWM with a two-phase "lub-dub"
  ramp pattern, rest period scaled by accelerometer movement score
- Configure LIS2DU12 wake-up-on-motion (INT2) and enter STM32
  Shutdown mode after a period of no movement
- Set unused GPIOs to analog mode before shutdown to eliminate
  floating-pin leakage
- Bump reverse-polarity protection gate resistor (R1) from 100k to
  2M on the PCB, cutting its static draw from 30uA to ~1.5uA
Parts:
- removed C1, C4: 10uF, Capacitor_SMD:C_0402_1005Metric
- added C10: 1uF, Capacitor_SMD:C_0603_1608Metric, F.Cu at (136.2, 91.5)
- added C11: 1uF, Capacitor_SMD:C_0603_1608Metric, F.Cu at (136.2, 93.5)
- C9: footprint Capacitor_SMD:C_0402_1005Metric -> Capacitor_SMD:C_0603_1608Metric
- R1: value 100k -> 10M

Commit message: -In progress porting code to LIS2DW12.
Parts:
- added R5: 0, Resistor_SMD:R_0402_1005Metric, F.Cu at (134.6, 100.8)
- TP4: footprint EN_Designs-Footprints:TestPoint_Pad_D0.5mm -> TestPoint:TestPoint_Pad_D1.0mm
- moved TP4 22.5 mm to (134.6, 98.3)
Connections:
- net Net-(U2-PF2) renamed /RST
Other:
- board text added: "V+"
- board text removed: "3V3"

Commit message: Changed optiisation, removed unused code, fixed bug of wrong flash size for KU4 chip
Parts:
- added TP10: TestPoint, TestPoint:TestPoint_Pad_D1.0mm, F.Cu at (130.0, 98.0)
- added TP15: TestPoint, EN_Designs-Footprints:TestPoint_Pad_D0.5mm, F.Cu at (136.6, 110.0)
- added TP4: TestPoint, EN_Designs-Footprints:TestPoint_Pad_D0.5mm, F.Cu at (136.6, 106.4)
- added TP5: TestPoint, EN_Designs-Footprints:TestPoint_Pad_D0.5mm, F.Cu at (136.6, 108.2)
- added TP6: TestPoint, EN_Designs-Footprints:TestPoint_Pad_D0.5mm, F.Cu at (134.8, 106.4)
- added TP7: TestPoint, EN_Designs-Footprints:TestPoint_Pad_D0.5mm, F.Cu at (134.8, 108.2)
- added TP8: TestPoint, EN_Designs-Footprints:TestPoint_Pad_D0.5mm, F.Cu at (134.8, 110.0)
- added TP9: TestPoint, EN_Designs-Footprints:TestPoint_Pad_D0.5mm, F.Cu at (134.8, 111.8)
- renumbered C11 to C1, C10 to C4, R5 to R1, R1 to R2, R2 to R3, R3 to R4, R4 to R5, TP4 to TP11, TP5 to TP12, TP6 to TP13, TP7 to TP14, TP8 to TP16
Connections:
- U2 pad 19: unconnected-(U2-PA9-Pad19) -> /TX

Commit message: -PCB jumper change
Parts:
- removed R1: 0, Resistor_SMD:R_0402_1005Metric
- added JP1: SolderJumper_2_Open, Jumper:SolderJumper-2_P1.3mm_Open_RoundedPad1.0x1.5mm, F.Cu at (146.8, 107.9)

Commit message: Improved error handling in LIS2 sleep function. Changed pulldowns Added jumpers to PCB
Parts:
- added JP2: SolderJumper_2_Bridged, Jumper:SolderJumper-2_P1.3mm_Bridged_RoundedPad1.0x1.5mm, F.Cu at (147.1, 112.7)
Connections:
- C1 pad 1: VCC -> Net-(JP2-B)
- C2 pad 1: VCC -> Net-(JP2-B)
- U1 pad 9: VCC -> Net-(JP2-B)
Routing:
- net VCC: track 19.1 -> 17.3 mm, vias 7 -> 6
- net Net-(JP2-B): track 0.00 -> 1.80 mm, vias 0 -> 1

Commit message: -changed accelerometer model
Parts:
- removed U1: LIS2DU12TR, EN_Designs-Footprints:LIS2DU12
- added REF**: BatteryHolder_LINX_BAT-HLD-012-SMT, Battery:BatteryHolder_LINX_BAT-HLD-012-SMT, B.Cu at (150.0, 90.0)
- added U3: LIS2DW12, EN_Designs-Footprints:LIS2DW12, F.Cu at (150.0, 95.5)
- R2: value 10M -> 20M
